File: Schematic/PiDuinoSerial/PiDuinoSerial.sch (EAGLE design)
At the start: 14 parts, among them IC1 ATMEGA8, J1 D0..D7, J2 Analogs, J3 D8_D13, Q1 16Mhz

Commit message: V0.05
Added Android java source code
Parts:
- added J4: PIPins8b, pinhead:PINHD-1X8
- added J5: PiPins8a, pinhead:PINHD-1X8
- added JP2: Pi4Pins, SparkFun-Connectors:M04PTH
Connections:
- new net N$10: J4.8, JP5.8
- new net N$11: J5.1, JP4.6
- new net N$12: J5.2, JP4.7
- new net N$13: J5.3, JP4.8
- new net N$14: J5.4, JP4.9
- new net N$15: J5.5, JP4.10
- new net N$16: J5.6, JP4.11
- new net N$17: J5.7, JP4.12
- new net N$18: J5.8, JP4.13
- new net N$19: JP2.1, JP4.5
- new net N$20: JP2.2, JP4.4
- new net N$21: JP2.3, JP4.3
- new net N$22: JP2.4, JP4.2
- new net N$3: J4.1, JP5.1
- new net N$4: J4.2, JP5.2
- new net N$5: J4.3, JP5.3
- new net N$6: J4.4, JP5.4
- new net N$7: J4.5, JP5.5
- new net N$8: J4.6, JP5.6
- new net N$9: J4.7, JP5.7
Changed lines of the file:
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@@
 <part name="GND7" library="SparkFun" deviceset="GND" device=""/>
 <part name="P+2" library="SparkFun" deviceset="VCC" device=""/>
+<part name="J4" library="pinhead" deviceset="PINHD-1X8" device="" value="PIPins8b"/>
+<part name="J5" library="pinhead" deviceset="PINHD-1X8" device="" value="PiPins8a"/>
+<part name="JP2" library="SparkFun-Connectors" deviceset="M04" device="PTH" value="Pi4Pins"/>
 </parts>
 <sheets>
@@
 <instance part="GND7" gate="1" x="-7.62" y="76.2" rot="R90"/>
 <instance part="P+2" gate="1" x="68.58" y="55.88"/>
+<instance part="J4" gate="A" x="45.72" y="111.76" rot="MR180"/>
+<instance part="J5" gate="A" x="3.81" y="109.22" rot="MR0"/>
+<instance part="JP2" gate="G$1" x="3.81" y="124.46"/>
 </instances>
 <busses>
@@
 </segment>
 </net>
+<net name="N$3" class="0">
+<segment>
+<pinref part="JP5" gate="G$1" pin="1"/>
+<pinref part="J4" gate="A" pin="1"/>
+<wire x1="43.18" y1="101.6" x2="35.56" y2="101.6" width="0.1524" layer="91"/>
+</segment>
+</net>
+<net name="N$4" class="0">
+<segment>
+<pinref part="JP5" gate="G$1" pin="2"/>
+<pinref part="J4" gate="A" pin="2"/>
+<wire x1="43.18" y1="104.14" x2="35.56" y2="104.14" width="0.1524" layer="91"/>
+</segment>
+</net>
+<net name="N$5" class="0">
+<segment>
+<pinref part="JP5" gate="G$1" pin="3"/>
+<pinref part="J4" gate="A" pin="3"/>
+<wire x1="43.18" y1="106.68" x2="35.56" y2="106.68" width="0.1524" layer="91"/>
+</segment>
+</net>
+<net name="N$6" class="0">
+<segment>
+<pinref part="JP5" gate="G$1" pin="4"/>
+<pinref part="J4" gate="A" pin="4"/>
+<wire x1="43.18" y1="109.22" x2="35.56" y2="109.22" width="0.1524" layer="91"/>
+</segment>
+</net>
+<net name="N$7" class="0">
+<segment>
+<pinref part="JP5" gate="G$1" pin="5"/>
+<pinref part="J4" gate="A" pin="5"/>
+<wire x1="43.18" y1="111.76" x2="35.56" y2="111.76" width="0.1524" layer="91"/>
+</segment>
+</net>
+<net name="N$8" class="0">
+<segment>
+<pinref part="JP5" gate="G$1" pin="6"/>
+<pinref part="J4" gate="A" pin="6"/>
+<wire x1="43.18" y1="114.3" x2="35.56" y2="114.3" width="0.1524" layer="91"/>
+</segment>
+</net>
+<net name="N$9" class="0">
+<segment>
+<pinref part="JP5" gate="G$1" pin="7"/>
+<pinref part="J4" gate="A" pin="7"/>
+<wire x1="43.18" y1="116.84" x2="35.56" y2="116.84" width="0.1524" layer="91"/>
+</segment>
+</net>
+<net name="N$10" class="0">
+<segment>
+<pinref part="JP5" gate="G$1" pin="8"/>
+<pinref part="J4" gate="A" pin="8"/>
+<wire x1="43.18" y1="119.38" x2="35.56" y2="119.38" width="0.1524" layer="91"/>
+</segment>
+</net>
+<net name="N$11" class="0">
+<segment>
+<pinref part="JP4" gate="G$1" pin="6"/>
+<pinref part="J5" gate="A" pin="1"/>
+<wire x1="6.35" y1="119.38" x2="12.7" y2="119.38" width="0.1524" layer="91"/>
+</segment>
+</net>
+<net name="N$12" class="0">
+<segment>
+<pinref part="JP4" gate="G$1" pin="7"/>
+<pinref part="J5" gate="A" pin="2"/>
+<wire x1="6.35" y1="116.84" x2="12.7" y2="116.84" width="0.1524" layer="91"/>
+</segment>
+</net>
+<net name="N$13" class="0">
+<segment>
+<pinref part="JP4" gate="G$1" pin="8"/>
+<pinref part="J5" gate="A" pin="3"/>
+<wire x1="6.35" y1="114.3" x2="12.7" y2="114.3" width="0.1524" layer="91"/>
+</segment>
+</net>
+<net name="N$14" class="0">
+<segment>
+<pinref part="JP4" gate="G$1" pin="9"/>
+<pinref part="J5" gate="A" pin="4"/>
+<wire x1="6.35" y1="111.76" x2="12.7" y2="111.76" width="0.1524" layer="91"/>
+</segment>
+</net>
+<net name="N$15" class="0">
+<segment>
+<pinref part="JP4" gate="G$1" pin="10"/>
+<pinref part="J5" gate="A" pin="5"/>
+<wire x1="6.35" y1="109.22" x2="12.7" y2="109.22" width="0.1524" layer="91"/>
+</segment>
+</net>
+<net name="N$16" class="0">
+<segment>
+<pinref part="JP4" gate="G$1" pin="11"/>
+<pinref part="J5" gate="A" pin="6"/>
+<wire x1="6.35" y1="106.68" x2="12.7" y2="106.68" width="0.1524" layer="91"/>
+</segment>
+</net>
+<net name="N$17" class="0">
+<segment>
+<pinref part="JP4" gate="G$1" pin="12"/>
+<pinref part="J5" gate="A" pin="7"/>
+<wire x1="6.35" y1="104.14" x2="12.7" y2="104.14" width="0.1524" layer="91"/>
+</segment>
+</net>
+<net name="N$18" class="0">
+<segment>
+<pinref part="JP4" gate="G$1" pin="13"/>
+<pinref part="J5" gate="A" pin="8"/>
+<wire x1="6.35" y1="101.6" x2="12.7" y2="101.6" width="0.1524" layer="91"/>
+</segment>
+</net>
+<net name="N$19" class="0">
+<segment>
+<pinref part="JP4" gate="G$1" pin="5"/>
+<pinref part="JP2" gate="G$1" pin="1"/>
+<wire x1="8.89" y1="121.92" x2="12.7" y2="121.92" width="0.1524" layer="91"/>
+</segment>
+</net>
+<net name="N$20" class="0">
+<segment>
+<pinref part="JP4" gate="G$1" pin="4"/>
+<pinref part="JP2" gate="G$1" pin="2"/>
+<wire x1="8.89" y1="124.46" x2="12.7" y2="124.46" width="0.1524" layer="91"/>
+</segment>
+</net>
+<net name="N$21" class="0">
+<segment>
+<pinref part="JP4" gate="G$1" pin="3"/>
+<pinref part="JP2" gate="G$1" pin="3"/>
+<wire x1="8.89" y1="127" x2="12.7" y2="127" width="0.1524" layer="91"/>
+</segment>
+</net>
+<net name="N$22" class="0">
+<segment>
+<pinref part="JP4" gate="G$1" pin="2"/>
+<pinref part="JP2" gate="G$1" pin="4"/>
+<wire x1="8.89" y1="129.54" x2="12.7" y2="129.54" width="0.1524" layer="91"/>
+</segment>
+</net>
