File: Schematic/RFHBridge/nRF24L01HBridge.brd (EAGLE design)
At the start: 49.2 x 44.5 mm, 20 parts, among them IC1 MEGA8-P, IC2 SN754410

Commit message: V0.05
Added Android java source code
Parts:
- removed JP1: HBridge, SparkFun:1X04
- removed JP4: BB, SparkFun:1X01
- added T1: 2N3565, transistor-neu-to92:TO92
Connections:
- removed net N$17: IC1.25, JP1.3
- removed net N$18: IC1.26, JP1.4
- removed net N$21: IC1.28, JP4.1
- new net D16: IC1.25
- new net D17: IC1.26, U$1.5
- new net D19: IC1.28
- new net N$9: JP14.3, T1.1
- net D18: no longer U$1.5
- net D2: no longer JP1.1
- net D3: now also T1.2; no longer JP14.3
- net D4: no longer JP1.2
- net GND: now also T1.3
Routing:
- net D4: track 29.1 -> 0.00 mm, vias 1 -> 0
- net D2: track 26.9 -> 0.00 mm, vias 1 -> 0
- net N$17: track 24.9 -> 0.00 mm, vias 1 -> 0
- net N$18: track 24.6 -> 0.00 mm, vias 1 -> 0
- net D12: track 68.9 -> 46.9 mm, vias 2 -> 1
- net D10: track 60.4 -> 39.1 mm, vias 0 -> 1
- net D17: track 0.00 -> 18.8 mm
- net D13: track 40.7 -> 54.3 mm
- net D18: track 13.5 -> 0.00 mm
- net D0: track 36.5 -> 25.1 mm
- net GND: track 172.3 -> 160.9 mm
- net D11: track 45.3 -> 55.9 mm
- net N$21: track 10.2 -> 0.00 mm
- net D3: track 53.3 -> 44.0 mm
- net 3.3V: track 72.4 -> 80.6 mm
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