File: Schematic/RFHBridge/nRF24L01HBridge.sch (EAGLE design)
At the start: 20 parts, among them IC1 MEGA8-P, IC2 SN754410

Commit message: V0.05
Added Android java source code
Parts:
- removed JP1: HBridge, SparkFun:M04PTH
- removed JP4: BB, SparkFun:M01PTH
- added T1: 2N3565, transistor-neu-to92:2N3565
Connections:
- removed net N$17: IC1.PC2(ADC2), JP1.3
- removed net N$18: IC1.PC3(ADC3), JP1.4
- removed net N$21: IC1.PC5(ADC5/SCL), JP4.1
- new net D16: IC1.PC2(ADC2)
- new net D17: IC1.PC3(ADC3), U$1.5
- new net D19: IC1.PC5(ADC5/SCL)
- new net N$9: JP14.3, T1.C
- net D18: no longer U$1.5
- net D2: no longer JP1.1
- net D3: now also T1.B; no longer JP14.3
- net D4: no longer JP1.2
- net GND: now also T1.E
Changed lines of the file:
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@@
 <part name="C1" library="SparkFun" deviceset="CAP_POL" device="PTH2" value="Cap nrf24l01"/>
 <part name="GND6" library="SparkFun" deviceset="GND" device=""/>
-<part name="JP1" library="SparkFun" deviceset="M04" device="PTH" value="HBridge"/>
 <part name="C2" library="SparkFun" deviceset="CAP" device="PTH" value="C1"/>
 <part name="C3" library="SparkFun" deviceset="CAP_POL" device="PTH1" value="C2"/>
@@
 <part name="GND2" library="SparkFun" deviceset="GND" device=""/>
 <part name="GND3" library="SparkFun" deviceset="GND" device=""/>
-<part name="JP4" library="SparkFun" deviceset="M01" device="PTH" value="BB"/>
 <part name="GND7" library="SparkFun" deviceset="GND" device=""/>
 <part name="GND8" library="SparkFun" deviceset="GND" device=""/>
@@
 <part name="JP3" library="SparkFun-Connectors" deviceset="M02" device="LOCK" value="Motor2"/>
 <part name="JP5" library="SparkFun-Connectors" deviceset="M01" device="PTH" value="MotorPower"/>
+<part name="T1" library="transistor-neu-to92" deviceset="2N3565" device=""/>
+<part name="GND12" library="SparkFun" deviceset="GND" device=""/>
 </parts>
 <sheets>
@@
 <instance part="JP15" gate="G$1" x="135.89" y="60.96" rot="R180"/>
 <instance part="P+5" gate="1" x="124.46" y="93.98" rot="R90"/>
-<instance part="GND4" gate="1" x="124.46" y="88.9"/>
+<instance part="GND4" gate="1" x="128.27" y="91.44" rot="R270"/>
 <instance part="P+6" gate="1" x="134.62" y="16.51" rot="R180"/>
 <instance part="U$1" gate="G$1" x="68.58" y="0"/>
@@
 <instance part="C1" gate="G$1" x="30.48" y="-25.4"/>
 <instance part="GND6" gate="1" x="30.48" y="-35.56"/>
-<instance part="JP1" gate="G$1" x="144.78" y="76.2" rot="R180"/>
 <instance part="C2" gate="G$1" x="25.4" y="43.18"/>
 <instance part="C3" gate="G$1" x="17.78" y="48.26"/>
@@
 <instance part="GND2" gate="1" x="25.4" y="35.56"/>
 <instance part="GND3" gate="1" x="17.78" y="40.64"/>
-<instance part="JP4" gate="G$1" x="114.3" y="66.04" rot="R180"/>
 <instance part="GND7" gate="1" x="86.36" y="-5.08"/>
 <instance part="GND8" gate="1" x="134.62" y="21.59" rot="R180"/>
@@
 <instance part="JP3" gate="G$1" x="-6.35" y="25.4" rot="R180"/>
 <instance part="JP5" gate="G$1" x="-17.78" y="6.35"/>
+<instance part="T1" gate="G$1" x="125.73" y="83.82"/>
+<instance part="GND12" gate="1" x="133.35" y="78.74" rot="R90"/>
 </instances>
 <busses>
@@
 </segment>
 <segment>
-<wire x1="138.43" y1="91.44" x2="124.46" y2="91.44" width="0.2032" layer="91"/>
+<wire x1="138.43" y1="91.44" x2="130.81" y2="91.44" width="0.2032" layer="91"/>
 <pinref part="JP14" gate="G$1" pin="2"/>
 <pinref part="GND4" gate="1" pin="GND"/>
@@
 <junction x="-36.83" y="7.62"/>
 </segment>
+<segment>
+<pinref part="T1" gate="G$1" pin="E"/>
+<pinref part="GND12" gate="1" pin="GND"/>
+<wire x1="130.81" y1="78.74" x2="128.27" y2="78.74" width="0.1524" layer="91"/>
+</segment>
 </net>
 <net name="VCC" class="0">
@@
 <pinref part="P+12" gate="1" pin="VCC"/>
 <wire x1="-39.37" y1="48.26" x2="-35.56" y2="48.26" width="0.1524" layer="91"/>
-</segment>
-</net>
-<net name="N$17" class="0">
-<segment>
-<wire x1="96.52" y1="73.66" x2="139.7" y2="73.66" width="0.2032" layer="91"/>
-<pinref part="IC1" gate="G$1" pin="PC2(ADC2)"/>
-<pinref part="JP1" gate="G$1" pin="3"/>
-</segment>
-</net>
-<net name="N$18" class="0">
-<segment>
-<wire x1="96.52" y1="71.12" x2="139.7" y2="71.12" width="0.2032" layer="91"/>
-<pinref part="IC1" gate="G$1" pin="PC3(ADC3)"/>
-<pinref part="JP1" gate="G$1" pin="4"/>
-</segment>
-</net>
-<net name="N$21" class="0">
-<segment>
-<wire x1="106.68" y1="66.04" x2="96.52" y2="66.04" width="0.1524" layer="91"/>
-<pinref part="IC1" gate="G$1" pin="PC5(ADC5/SCL)"/>
-<pinref part="JP4" gate="G$1" pin="1"/>
 </segment>
 </net>
@@
 </segment>
 <segment>
-<wire x1="138.43" y1="88.9" x2="132.08" y2="88.9" width="0.1524" layer="91"/>
-<label x="132.08" y="88.9" size="1.778" layer="95"/>
-<pinref part="JP14" gate="G$1" pin="3"/>
+<pinref part="T1" gate="G$1" pin="B"/>
+<wire x1="123.19" y1="83.82" x2="118.11" y2="83.82" width="0.1524" layer="91"/>
+<label x="118.11" y="83.82" size="1.778" layer="95"/>
 </segment>
 </net>
@@
 <pinref part="IC1" gate="G$1" pin="PD4(XCK/T0)"/>
 </segment>
-<segment>
-<wire x1="139.7" y1="76.2" x2="127" y2="76.2" width="0.1524" layer="91"/>
-<label x="127" y="76.2" size="1.778" layer="95"/>
-<pinref part="JP1" gate="G$1" pin="2"/>
-</segment>
 </net>
 <net name="D2" class="0">
@@
 <label x="102.87" y="50.8" size="1.778" layer="95"/>
 <pinref part="IC1" gate="G$1" pin="PD2(INT0)"/>
-</segment>
-<segment>
-<wire x1="139.7" y1="78.74" x2="133.35" y2="78.74" width="0.1524" layer="91"/>
-<label x="133.35" y="78.74" size="1.778" layer="95"/>
-<pinref part="JP1" gate="G$1" pin="1"/>
 </segment>
 </net>
@@
 <pinref part="IC1" gate="G$1" pin="PC4(ADC4/SDA)"/>
 </segment>
-<segment>
-<wire x1="60.96" y1="0" x2="50.8" y2="0" width="0.1524" layer="91"/>
-<label x="50.8" y="0" size="1.778" layer="95"/>
-<pinref part="U$1" gate="G$1" pin="5"/>
-</segment>
 </net>
 <net name="D14" class="0">
@@
 </segment>
 </net>
+<net name="D17" class="0">
+<segment>
+<pinref part="U$1" gate="G$1" pin="5"/>
+<wire x1="60.96" y1="0" x2="54.61" y2="0" width="0.1524" layer="91"/>
+<label x="54.61" y="0" size="1.778" layer="95"/>
+</segment>
+<segment>
+<pinref part="IC1" gate="G$1" pin="PC3(ADC3)"/>
+<wire x1="96.52" y1="71.12" x2="102.87" y2="71.12" width="0.1524" layer="91"/>
+<label x="102.87" y="71.12" size="1.778" layer="95"/>
+</segment>
+</net>
+<net name="D16" class="0">
+<segment>
+<pinref part="IC1" gate="G$1" pin="PC2(ADC2)"/>
+<wire x1="96.52" y1="73.66" x2="102.87" y2="73.66" width="0.1524" layer="91"/>
+<label x="102.87" y="73.66" size="1.778" layer="95"/>
+</segment>
+</net>
+<net name="D19" class="0">
+<segment>
+<pinref part="IC1" gate="G$1" pin="PC5(ADC5/SCL)"/>
+<wire x1="96.52" y1="66.04" x2="102.87" y2="66.04" width="0.1524" layer="91"/>
+<label x="102.87" y="66.04" size="1.778" layer="95"/>
+</segment>
+</net>
+<net name="N$9" class="0">
+<segment>
+<pinref part="JP14" gate="G$1" pin="3"/>
+<pinref part="T1" gate="G$1" pin="C"/>
+<wire x1="128.27" y1="88.9" x2="138.43" y2="88.9" width="0.1524" layer="91"/>
+</segment>
+</net>
